File: small-fry-pcb.sch (KiCad schematic (older format))
At the start: 139 parts, among them U1 STM32F303CCT6

Commit message: updated schematic and fixed footprints
Parts:
- MX1, MX10, MX2, MX3, MX4, MX5, MX6, MX7, MX8, MX9: footprint Keebio-Parts:MX-Alps-Choc-1U -> MX_Alps_Hybrid:MX-1.75U-NoLED
- MX11, MX12, MX13, MX14, MX15, MX16, MX17, MX18, MX19, MX20, MX21, MX22, MX23, MX24, MX26, MX27, MX28, MX29, MX31, MX32, MX33, MX34, MX35, MX36, MX37, MX38, MX39, MX40, MX41, MX42, MX43, MX44, MX45, MX46, MX47, MX48, MX49, MX50, MX51, MX52, MX53, MX54, MX55, MX56, MX57, MX58, MX59, MX60, MX61, MX62, MX63, MX64, MX65, MX66, MX67, MX68, MX69: footprint Keebio-Parts:MX-Alps-Choc-1U -> MX_Alps_Hybrid:MX-1U-NoLED
- MX25: footprint Keebio-Parts:MX-Alps-Choc-1U -> MX_Alps_Hybrid:MX-2.25U-ReversedStabilizers-NoLED
- MX30: footprint Keebio-Parts:MX-Alps-Choc-1U -> MX_Alps_Hybrid:MX-2.75U-ReversedStabilizers-NoLED
