File: small-fry-pcb.kicad_pcb (KiCad board)
At the start: 2 copper layers, 138 parts

Commit message: Squashed commit of the following:
commit 3a31e5c864698379eab5fa9799b6646026e60a6b
Author: anchovie-codes <littlebrother.free@gmail.com>
Date:   Mon Sep 2 00:25:19 2024 -0400

    backup file changes

commit 27ca4d82953605882c5c8308233a3a86d2bdc34d
Author: anchovie-codes <littlebrother.free@gmail.com>
Date:   Mon Sep 2 00:24:05 2024 -0400

    so much rerouting

commit 9fd5b48f56c3140a57fcb4215c1e2a66e7782bf8
Author: anchovie-codes <littlebrother.free@gmail.com>
Date:   Sun Sep 1 19:36:35 2024 -0400

    added new logo

commit 6d58b5c3b37e970dc2157a1aee4402dd0390434d
Author: anchovie-codes <littlebrother.free@gmail.com>
Date:   Sun Sep 1 18:15:21 2024 -0400

    added slikscreen

commit eb283958132534611e3bdf4a2205f7fc4c43aa94
Author: anchovie-codes <littlebrother.free@gmail.com>
Date:   Sun Sep 1 15:57:01 2024 -0400

    finished first attempt routing

commit ba8867c2d6ba6c449a2bbe37d6967075e8a42684
Author: anchovie-codes <littlebrother.free@gmail.com>
Date:   Sun Sep 1 12:28:37 2024 -0400

    replaced bonsai with pico
Parts:
- added G***: LOGO, LOGO, F.Cu at (43.0, 106.0)
- added G***: LOGO, LOGO, F.Cu at (373.0, 96.0)
- added G***: LOGO, LOGO, B.Cu at (201.0, 77.0)
- added U1: Pico, MCU_RaspberryPi_and_Boards:RPi_Pico_SMD_TH, F.Cu at (43.4, 54.5)
- D1, D10, D11, D12, D13, D14, D15, D16, D17, D18, D19, D2, D20, D21, D22, D23, D24, D25, D26, D27, D28, D29, D3, D30, D31, D32, D33, D34, D35, D36, D37, D38, D39, D4, D40, D41, D42, D43, D44, D45, D46, D47, D48, D49, D5, D50, D51, D52, D53, D54, D55, D56, D57, D58, D59, D6, D60, D61, D62, D63, D64, D65, D66, D67, D68, D69, D7, D8, D9: moved to B.Cu
- MX10, MX3, MX4, MX5, MX6, MX7, MX8, MX9: footprint MX_Alps_Hybrid:MX-1.75U-NoLED -> MX_Alps_Hybrid:MX-1U-NoLED
- MX15, MX16, MX17, MX31, MX32, MX44, MX45, MX46, MX57, MX58, MX59: footprint MX_Alps_Hybrid:MX-1U-NoLED -> MX_Alps_Hybrid:MX-1.75U-NoLED
- MX25: footprint MX_Alps_Hybrid:MX-2.25U-ReversedStabilizers-NoLED -> MX_Alps_Hybrid:MX-1U-NoLED
- MX30: footprint MX_Alps_Hybrid:MX-2.75U-ReversedStabilizers-NoLED -> MX_Alps_Hybrid:MX-1.75U-NoLED
- MX62: footprint MX_Alps_Hybrid:MX-1U-NoLED -> MX_Alps_Hybrid:MX-2.25U-ReversedStabilizers-NoLED
- MX63: footprint MX_Alps_Hybrid:MX-1U-NoLED -> MX_Alps_Hybrid:MX-2.75U-ReversedStabilizers-NoLED
- moved D30 357.5 mm to (372.5, 62.9)
- moved D69 334.7 mm to (370.1, 124.8)
- moved D15 331.6 mm to (372.5, 43.8)
- moved MX30 322.0 mm to (372.5, 57.9)
- moved D14 312.4 mm to (346.3, 43.8)
- moved D68 301.6 mm to (351.1, 124.8)
- moved D13 293.9 mm to (327.3, 43.8)
- moved D12 282.7 mm to (308.2, 43.8)
- moved D29 280.6 mm to (346.3, 62.9)
- moved D57 275.4 mm to (334.4, 101.0)
- moved D11 269.8 mm to (289.2, 43.8)
- moved D28 266.3 mm to (327.3, 62.9)
- moved D27 265.6 mm to (308.2, 62.9)
- moved MX69 263.7 mm to (370.1, 119.8)
- moved D67 254.7 mm to (332.0, 124.8)
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Connections:
- D10 pad 1: row4 -> row0
- D12 pad 1: row1 -> row0
- D13 pad 1: row2 -> row0
- D14 pad 1: row3 -> row0
- D15 pad 1: row4 -> row0
- D16 pad 1: row0 -> row1
- D18 pad 1: row2 -> row1
- D19 pad 1: row3 -> row1
- D2 pad 1: row1 -> row0
- D20 pad 1: row4 -> row1
- D21 pad 1: row0 -> row1
- D23 pad 1: row2 -> row1
- D24 pad 1: row3 -> row1
- D25 pad 1: row4 -> row1
- D26 pad 1: row0 -> row1
- D28 pad 1: row2 -> row1
- D29 pad 1: row3 -> row1
- D3 pad 1: row2 -> row0
- D30 pad 1: row4 -> row1
- D31 pad 1: row0 -> row2
- D32 pad 1: row1 -> row2
- D34 pad 1: row3 -> row2
- D35 pad 1: row4 -> row2
- D36 pad 1: row0 -> row2
- D37 pad 1: row1 -> row2
- D39 pad 1: row3 -> row2
- D4 pad 1: row3 -> row0
- D40 pad 1: row4 -> row2
- D41 pad 1: row0 -> row2
- D42 pad 1: row1 -> row2
- D44 pad 1: row3 -> row2
- D45 pad 1: row0 -> row3
- D46 pad 1: row1 -> row3
- D47 pad 1: row2 -> row3
- D48 pad 1: row4 -> row3
- D5 pad 1: row4 -> row0
- D50 pad 1: row0 -> row3
- D51 pad 1: row1 -> row3
- D52 pad 1: row2 -> row3
- D53 pad 1: row4 -> row3
- D55 pad 1: row0 -> row3
- D56 pad 1: row1 -> row3
- D57 pad 1: row2 -> row3
- D59 pad 1: row3 -> row4
- D60 pad 1: row0 -> row4
- D61 pad 1: row1 -> row4
- D62 pad 1: row2 -> row4
- D64 pad 1: row3 -> row4
- D65 pad 1: row0 -> row4
- D66 pad 1: row1 -> row4
- D67 pad 1: row2 -> row4
- D68 pad 1: row0 -> row4
- D69 pad 1: row1 -> row4
- D7 pad 1: row1 -> row0
- D8 pad 1: row2 -> row0
- D9 pad 1: row3 -> row0
- MX10 pad 1: col1 -> col9
- MX11 pad 1: col2 -> col10
- MX12 pad 1: col2 -> col11
- MX13 pad 1: col2 -> col12
- MX14 pad 1: col2 -> col13
- MX15 pad 1: col2 -> col14
- MX16 pad 1: col3 -> col0
- MX17 pad 1: col3 -> col1
- MX18 pad 1: col3 -> col2
- MX2 pad 1: col0 -> col1
- MX20 pad 1: col3 -> col4
- MX21 pad 1: col4 -> col5
- MX22 pad 1: col4 -> col6
- MX23 pad 1: col4 -> col7
- MX24 pad 1: col4 -> col8
- MX25 pad 1: col4 -> col9
- MX26 pad 1: col5 -> col10
- MX27 pad 1: col5 -> col11
- MX28 pad 1: col5 -> col12
- MX29 pad 1: col5 -> col13
- MX3 pad 1: col0 -> col2
- MX30 pad 1: col5 -> col14
- MX31 pad 1: col6 -> col0
- MX32 pad 1: col6 -> col1
- MX33 pad 1: col6 -> col2
- MX34 pad 1: col6 -> col3
- MX35 pad 1: col6 -> col4
- MX36 pad 1: col7 -> col5
- MX37 pad 1: col7 -> col6
- MX39 pad 1: col7 -> col8
- MX4 pad 1: col0 -> col3
- MX40 pad 1: col7 -> col9
- MX41 pad 1: col8 -> col10
- MX42 pad 1: col8 -> col11
- MX43 pad 1: col8 -> col12
- MX44 pad 1: col8 -> col13
- MX45 pad 1: col9 -> col0
- MX46 pad 1: Net-(MX46-Pad1) -> col1
- MX47 pad 1: Net-(MX46-Pad1) -> col2
- MX48 pad 1: col8 -> col3
- MX49 pad 1: Net-(MX46-Pad1) -> col4
- MX5 pad 1: col0 -> col4
- MX50 pad 1: col10 -> col5
- MX51 pad 1: col10 -> col6
- MX52 pad 1: col10 -> col7
- MX53 pad 1: Net-(MX46-Pad1) -> col8
- MX54 pad 1: col10 -> col9
- MX55 pad 1: col11 -> col10
- MX57 pad 1: col11 -> col12
- MX58 pad 1: col10 -> col0
- MX59 pad 1: col11 -> col1
- MX6 pad 1: col1 -> col5
- MX60 pad 1: col12 -> col2
- MX61 pad 1: col12 -> col3
- MX62 pad 1: col12 -> col4
- MX63 pad 1: col11 -> col5
- MX64 pad 1: col12 -> col6
- MX65 pad 1: col13 -> col7
- MX66 pad 1: col13 -> col8
- MX67 pad 1: col13 -> col9
- MX68 pad 1: col14 -> col10
- MX69 pad 1: col14 -> col11
- MX7 pad 1: col1 -> col6
- MX8 pad 1: col1 -> col7
- MX9 pad 1: col1 -> col8
Routing:
- net col12: track 0.00 -> 723.1 mm
- net col11: track 0.00 -> 711.2 mm
- net col10: track 0.00 -> 685.8 mm
- net col13: track 0.00 -> 655.3 mm
- net col8: track 0.00 -> 606.7 mm
- net col7: track 0.00 -> 582.4 mm
- net col14: track 0.00 -> 577.9 mm
- net col9: track 0.00 -> 567.5 mm
- net col6: track 0.00 -> 562.2 mm
- net col4: track 0.00 -> 513.1 mm
- net col5: track 0.00 -> 511.6 mm
- net col3: track 0.00 -> 466.6 mm
- net col2: track 0.00 -> 451.8 mm
- net row4: track 0.00 -> 449.8 mm, vias 0 -> 1
- net row0: track 0.00 -> 438.7 mm, vias 0 -> 1
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Other:
- board outline added: 370 x 103 mm
- net class Default removed
- rule pad_to_mask_clearance: 0.2 -> 0
- board text added: "GP15"
- board text added: "https://anchovie.art"

Commit message: updated matrix routing
Parts:
- removed the G*** at (201.0, 77.0)
- moved G*** 12.2 mm to (50.0, 96.0)
- moved D43 10.6 mm to (337.3, 78.3), turned to 90 degrees
- moved D28 10.6 mm to (337.3, 59.3), turned to 90 degrees
- moved D13 10.6 mm to (337.3, 40.2), turned to 90 degrees
- moved D68 10.6 mm to (361.1, 121.2), turned to 90 degrees
- moved D37 10.6 mm to (223.0, 78.3), turned to 90 degrees
- moved D22 10.6 mm to (223.0, 59.3), turned to 90 degrees
- moved D51 10.6 mm to (223.0, 97.4), turned to 90 degrees
- moved D7 10.6 mm to (223.0, 40.2), turned to 90 degrees
- moved D31 10.6 mm to (87.2, 78.3), turned to 90 degrees
- moved D32 10.6 mm to (120.6, 78.3), turned to 90 degrees
- moved D33 10.6 mm to (146.8, 78.3), turned to 90 degrees
- moved D34 10.6 mm to (165.8, 78.3), turned to 90 degrees
- moved D35 10.6 mm to (184.9, 78.3), turned to 90 degrees
- moved D36 10.6 mm to (203.9, 78.3), turned to 90 degrees
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Connections:
- MX63 pad 1: col5 -> col7
- MX64 pad 1: col6 -> col9
- MX65 pad 1: col7 -> col10
- MX66 pad 1: col8 -> col11
- MX67 pad 1: col9 -> col12
- MX68 pad 1: col10 -> col13
- MX69 pad 1: col11 -> col14
- U1 pad 1: row4 -> col14
- U1 pad 10: col13 -> col7
- U1 pad 11: col12 -> col6
- U1 pad 12: col11 -> col5
- U1 pad 14: col10 -> col4
- U1 pad 15: unconnected-(U1-GPIO11-Pad15) -> col3
- U1 pad 16: unconnected-(U1-GPIO12-Pad16) -> col2
- U1 pad 17: unconnected-(U1-GPIO13-Pad17) -> col1
- U1 pad 19: unconnected-(U1-GPIO14-Pad19) -> col0
- U1 pad 2: row3 -> col13
- U1 pad 21: col9 -> unconnected-(U1-GPIO16-Pad21)
- U1 pad 22: col8 -> row4
- U1 pad 24: col7 -> row3
- U1 pad 25: col6 -> row2
- U1 pad 26: col5 -> row1
- U1 pad 27: col4 -> row0
- U1 pad 29: col3 -> unconnected-(U1-GPIO22-Pad29)
- U1 pad 31: col2 -> unconnected-(U1-GPIO26_ADC0-Pad31)
- U1 pad 32: col1 -> unconnected-(U1-GPIO27_ADC1-Pad32)
- U1 pad 34: col0 -> unconnected-(U1-GPIO28_ADC2-Pad34)
- U1 pad 4: row2 -> col12
- U1 pad 5: row1 -> col11
- U1 pad 6: row0 -> col10
- U1 pad 7: unconnected-(U1-GPIO5-Pad7) -> col9
- U1 pad 9: col14 -> col8
Routing:
- net col10: track 685.8 -> 411.0 mm
- net col11: track 711.2 -> 444.1 mm
- net col12: track 723.1 -> 469.2 mm
- net col6: track 562.2 -> 314.6 mm
- net col0: track 390.5 -> 146.3 mm
- net col8: track 606.7 -> 366.0 mm
- net col7: track 582.4 -> 343.5 mm
- net col1: track 427.4 -> 190.4 mm
- net col2: track 451.8 -> 221.0 mm
- net col4: track 513.1 -> 282.9 mm
- net col3: track 466.6 -> 243.2 mm
- net col5: track 511.6 -> 304.1 mm
- net col9: track 567.5 -> 388.2 mm
- net col13: track 655.3 -> 493.6 mm
- net row0: track 438.7 -> 333.2 mm, vias 1 -> 0
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Other:
- board size 370 x 103 mm -> 365 x 103 mm

Commit message: adjusted col traces and silkscreen
Routing:
- net col0: track 146.3 -> 151.5 mm
- net col13: track 493.6 -> 498.7 mm
- net col11: track 444.1 -> 449.3 mm
- net col10: track 411.0 -> 416.2 mm
- net col5: track 304.1 -> 309.2 mm
- net col7: track 343.5 -> 348.6 mm
- net col1: track 190.4 -> 195.5 mm
- net col3: track 243.2 -> 248.3 mm
- net col6: track 314.6 -> 319.7 mm
- net col4: track 282.9 -> 288.1 mm
- net col2: track 221.0 -> 226.1 mm
- net col12: track 469.2 -> 474.3 mm
- net col9: track 388.2 -> 393.3 mm
- net col8: track 366.0 -> 371.1 mm
- net col14: track 513.9 -> 518.9 mm

Commit message: added extra switches
to accommodate the switch holes, leftmost diodes were moved and col routing was modified. extra pads connect back to the diodes.
Parts:
- added MX70: MX-NoLED, MX_Alps_Hybrid:MX-1.5U-NoLED, F.Cu at (81.6, 115.5)
- added MX71: MX-NoLED, MX_Alps_Hybrid:MX-1.5U-NoLED, F.Cu at (81.6, 96.4)
- added MX72: MX-NoLED, MX_Alps_Hybrid:MX-1.5U-NoLED, F.Cu at (81.6, 77.3)
- added MX73: MX-NoLED, MX_Alps_Hybrid:MX-1.5U-NoLED, F.Cu at (81.6, 58.3)
- added MX74: MX-NoLED, MX_Alps_Hybrid:MX-1.5U-NoLED, F.Cu at (81.6, 39.2)
- added MX75: MX-NoLED, MX_Alps_Hybrid:MX-1.5U-NoLED, F.Cu at (334.0, 96.4)
- added MX76: MX-NoLED, MX_Alps_Hybrid:MX-1.5U-NoLED, F.Cu at (353.1, 77.3)
- added MX77: MX-NoLED, MX_Alps_Hybrid:MX-1.5U-NoLED, F.Cu at (372.1, 58.3)
- added MX78: MX-NoLED, MX_Alps_Hybrid:MX-1.5U-NoLED, F.Cu at (372.1, 39.2)
- moved D16 16.2 mm to (71.0, 59.2)
- moved D1 16.2 mm to (71.0, 40.2)
- moved D31 16.2 mm to (71.0, 78.3)
- moved D45 16.2 mm to (71.0, 97.4)
- moved D58 16.2 mm to (71.0, 116.5)
Routing:
- net col14: track 518.9 -> 543.7 mm
- net Net-(D1-A): track 7.17 -> 24.2 mm
- net Net-(D58-A): track 7.09 -> 23.4 mm
- net col12: track 474.3 -> 490.3 mm
- net col13: track 498.7 -> 514.7 mm
- net Net-(D45-A): track 7.09 -> 22.2 mm
- net Net-(D31-A): track 7.09 -> 22.1 mm
- net Net-(D16-A): track 7.09 -> 22.1 mm
- net row0: track 333.2 -> 340.4 mm
- net col0: track 151.5 -> 158.1 mm
- net Net-(D57-A): track 7.09 -> 13.6 mm
- net Net-(D15-A): track 7.09 -> 13.5 mm
- net Net-(D30-A): track 7.09 -> 13.4 mm
- net Net-(D44-A): track 7.09 -> 13.4 mm
- net row4: track 358.6 -> 360.5 mm
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