File: small-fry-pcb.kicad_pcb (KiCad board)
At the start: 2 copper layers, 370 x 103 mm, 142 parts, among them U1 Pico

Commit message: Squashed commit of the following:
commit 176f3bbe4c1d8503f8e6634e84449ff57851d2da
Author: anchovie-codes <littlebrother.free@gmail.com>
Date:   Wed Sep 4 12:11:39 2024 -0400

    updated backup

commit faa0e4d37d006ebb0d8ebb4d260e99f9d3fc7be4
Author: anchovie-codes <littlebrother.free@gmail.com>
Date:   Wed Sep 4 12:06:31 2024 -0400

    adjusted col traces and silkscreen

commit 79d5b3e19d1111bf43eaceb8324e875e345697d4
Author: anchovie-codes <littlebrother.free@gmail.com>
Date:   Wed Sep 4 11:57:08 2024 -0400

    updated matrix routing
Parts:
- removed the G*** at (201.0, 77.0)
- moved G*** 12.2 mm to (50.0, 96.0)
- moved D43 10.6 mm to (337.3, 78.3), turned to 90 degrees
- moved D28 10.6 mm to (337.3, 59.3), turned to 90 degrees
- moved D13 10.6 mm to (337.3, 40.2), turned to 90 degrees
- moved D68 10.6 mm to (361.1, 121.2), turned to 90 degrees
- moved D37 10.6 mm to (223.0, 78.3), turned to 90 degrees
- moved D22 10.6 mm to (223.0, 59.3), turned to 90 degrees
- moved D51 10.6 mm to (223.0, 97.4), turned to 90 degrees
- moved D7 10.6 mm to (223.0, 40.2), turned to 90 degrees
- moved D31 10.6 mm to (87.2, 78.3), turned to 90 degrees
- moved D32 10.6 mm to (120.6, 78.3), turned to 90 degrees
- moved D33 10.6 mm to (146.8, 78.3), turned to 90 degrees
- moved D34 10.6 mm to (165.8, 78.3), turned to 90 degrees
- moved D35 10.6 mm to (184.9, 78.3), turned to 90 degrees
- moved D36 10.6 mm to (203.9, 78.3), turned to 90 degrees
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Connections:
- MX63 pad 1: col5 -> col7
- MX64 pad 1: col6 -> col9
- MX65 pad 1: col7 -> col10
- MX66 pad 1: col8 -> col11
- MX67 pad 1: col9 -> col12
- MX68 pad 1: col10 -> col13
- MX69 pad 1: col11 -> col14
- U1 pad 1: row4 -> col14
- U1 pad 10: col13 -> col7
- U1 pad 11: col12 -> col6
- U1 pad 12: col11 -> col5
- U1 pad 14: col10 -> col4
- U1 pad 15: unconnected-(U1-GPIO11-Pad15) -> col3
- U1 pad 16: unconnected-(U1-GPIO12-Pad16) -> col2
- U1 pad 17: unconnected-(U1-GPIO13-Pad17) -> col1
- U1 pad 19: unconnected-(U1-GPIO14-Pad19) -> col0
- U1 pad 2: row3 -> col13
- U1 pad 21: col9 -> unconnected-(U1-GPIO16-Pad21)
- U1 pad 22: col8 -> row4
- U1 pad 24: col7 -> row3
- U1 pad 25: col6 -> row2
- U1 pad 26: col5 -> row1
- U1 pad 27: col4 -> row0
- U1 pad 29: col3 -> unconnected-(U1-GPIO22-Pad29)
- U1 pad 31: col2 -> unconnected-(U1-GPIO26_ADC0-Pad31)
- U1 pad 32: col1 -> unconnected-(U1-GPIO27_ADC1-Pad32)
- U1 pad 34: col0 -> unconnected-(U1-GPIO28_ADC2-Pad34)
- U1 pad 4: row2 -> col12
- U1 pad 5: row1 -> col11
- U1 pad 6: row0 -> col10
- U1 pad 7: unconnected-(U1-GPIO5-Pad7) -> col9
- U1 pad 9: col14 -> col8
Routing:
- net col10: track 685.8 -> 416.2 mm
- net col11: track 711.2 -> 449.3 mm
- net col12: track 723.1 -> 474.3 mm
- net col6: track 562.2 -> 319.7 mm
- net col0: track 390.5 -> 151.5 mm
- net col8: track 606.7 -> 371.1 mm
- net col7: track 582.4 -> 348.6 mm
- net col1: track 427.4 -> 195.5 mm
- net col2: track 451.8 -> 226.1 mm
- net col4: track 513.1 -> 288.1 mm
- net col3: track 466.6 -> 248.3 mm
- net col5: track 511.6 -> 309.2 mm
- net col9: track 567.5 -> 393.3 mm
- net col13: track 655.3 -> 498.7 mm
- net row0: track 438.7 -> 333.2 mm, vias 1 -> 0
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Other:
- board size 370 x 103 mm -> 365 x 103 mm

Commit message: generated gerbers
Parts:
- added G***: LOGO, LOGO, F.Cu at (373.0, 98.0)
- G***: moved to B.Cu
- turned G*** to 180 degrees
Other:
- outline, holes or cut-outs redrawn

Commit message: changed mods, changed col stagger
Parts:
- removed the G*** at (50.0, 96.0)
- removed the G*** at (373.0, 98.0) (x2)
- added G***: LOGO, LOGO, F.Cu at (335.5, 91.0)
- added G***: LOGO, LOGO, F.Cu at (33.0, 92.5)
- added G***: LOGO, LOGO, B.Cu at (33.0, 92.5)
- added G***: LOGO, LOGO, B.Cu at (335.5, 91.0)
- MX1, MX16, MX31, MX45, MX58: footprint MX_Alps_Hybrid:MX-1.75U-NoLED -> MX_Alps_Hybrid:MX-1.25U-NoLED
- MX15, MX17, MX2, MX30, MX32, MX44, MX46, MX57, MX59: footprint MX_Alps_Hybrid:MX-1.75U-NoLED -> MX_Alps_Hybrid:MX-1.5U-NoLED
- moved D15 34.0 mm to (348.5, 39.1)
- moved D30 34.0 mm to (348.5, 58.1)
- moved D44 34.0 mm to (329.5, 77.2)
- moved D57 34.0 mm to (310.4, 96.2)
- moved MX15 34.0 mm to (340.5, 38.1)
- moved MX30 34.0 mm to (340.5, 57.1)
- moved MX44 34.0 mm to (321.5, 76.2)
- moved MX57 34.0 mm to (302.4, 95.2)
- moved D11 31.6 mm to (267.6, 39.1)
- moved D12 31.6 mm to (286.6, 39.1)
- moved D13 31.6 mm to (305.7, 39.1)
- moved D22 31.6 mm to (191.4, 58.1)
- moved D26 31.6 mm to (267.6, 58.1)
- moved D27 31.6 mm to (286.6, 58.1)
- moved D28 31.6 mm to (305.7, 58.1)
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Connections:
- MX62 pad 1: col4 -> col5
- MX63 pad 1: col7 -> col8
Routing:
- net col4: track 288.1 -> 252.1 mm
- net col5: track 309.2 -> 275.9 mm
- net col2: track 226.1 -> 201.0 mm
- net col3: track 248.3 -> 223.9 mm
- net col14: track 518.9 -> 494.7 mm
- net col8: track 371.1 -> 347.9 mm
- net col12: track 474.3 -> 451.7 mm
- net col7: track 348.6 -> 326.1 mm
- net col1: track 195.5 -> 173.4 mm
- net col13: track 498.7 -> 477.1 mm
- net col11: track 449.3 -> 430.6 mm
- net col10: track 416.2 -> 398.1 mm
- net col9: track 393.3 -> 375.5 mm
- net row1: track 326.3 -> 309.2 mm
- net col6: track 319.7 -> 303.3 mm
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Other:
- board size 365 x 103 mm -> 343 x 101 mm
- board text added: "rev. 2 by anchovie uwu https://anchovie.art"
- board text removed: "https://anchovie.art"

Commit message: changed footprints, rerouted
Parts:
- MX1, MX16, MX31, MX45, MX58: footprint MX_Alps_Hybrid:MX-1.25U-NoLED -> marbastlib-mx:SW_MX_1.25u
- MX10, MX11, MX12, MX13, MX14, MX18, MX19, MX20, MX21, MX22, MX23, MX24, MX25, MX26, MX27, MX28, MX29, MX3, MX33, MX34, MX35, MX36, MX37, MX38, MX39, MX4, MX40, MX41, MX42, MX43, MX47, MX48, MX49, MX5, MX50, MX51, MX52, MX53, MX54, MX55, MX56, MX6, MX60, MX61, MX64, MX65, MX66, MX67, MX68, MX69, MX7, MX8, MX9: footprint MX_Alps_Hybrid:MX-1U-NoLED -> marbastlib-mx:SW_MX_1u
- MX15, MX17, MX2, MX30, MX32, MX44, MX46, MX57, MX59: footprint MX_Alps_Hybrid:MX-1.5U-NoLED -> marbastlib-mx:SW_MX_1.5u
- MX62: footprint MX_Alps_Hybrid:MX-2.25U-ReversedStabilizers-NoLED -> MX_Solderable:MX-Solderable-2.25U-ReversedStabilizers
- MX63: footprint MX_Alps_Hybrid:MX-2.75U-ReversedStabilizers-NoLED -> MX_Solderable:MX-Solderable-2.75U-ReversedStabilizers
- moved G*** 3.50 mm to (332.0, 91.0) (x2)
Routing:
- net col8: track 347.9 -> 339.6 mm
- net col7: track 326.1 -> 321.4 mm
- net col6: track 303.3 -> 298.7 mm
- net col3: track 223.9 -> 228.3 mm
- net col2: track 201.0 -> 205.4 mm
- net col0: track 141.1 -> 145.2 mm
- net col1: track 173.4 -> 177.6 mm
- net col4: track 252.1 -> 248.1 mm
- net col14: track 494.7 -> 497.9 mm
- net col5: track 275.9 -> 273.2 mm
- net col11: track 430.6 -> 428.6 mm
- net col9: track 375.5 -> 373.6 mm
- net col10: track 398.1 -> 396.3 mm
Other:
- board size 343 x 101 mm -> 338.4 x 100.6 mm
